Commit message: Created separate copernicus sim folders to modularize the package

File: copernicus_sim/urdf/accessories/imu_copernicus.urdf.xacro (robot description, xacro)
@@ -25,5 +25,5 @@
 -->
 <robot name="copernicus" xmlns:xacro="https://ros.org/wiki/xacro">
-    <xacro:macro name="imu" params="frame:=imu topic:=imu/data update_rate:=20 robot_namespace:=/">
+    <xacro:macro name="imu" params="frame:=imu topic:=imu/data update_rate:=20 robot_namespace:=/ sim_type:=gazebo">
         <joint name="${frame}_joint" type="fixed">
             <parent link="base_link" />
@@ -38,23 +38,40 @@
             </inertial>
         </link>
-        <gazebo reference="${frame}">
-            <gravity>true</gravity>
-            <sensor name="imu_sensor" type="imu">
-                <always_on>true</always_on>
-                <update_rate>100</update_rate>
-                <visualize>true</visualize>
-                <topic>${topic}</topic>
-                <plugin filename="libgazebo_ros_imu_sensor.so" name="imu_plugin">
-                    <topicName>${topic}</topicName>
-                    <bodyName>${frame}</bodyName>
-                    <updateRateHZ>${update_rate}</updateRateHZ>
-                    <gaussianNoise>0.0</gaussianNoise>
-                    <xyzOffset>0 0 0</xyzOffset>
-                    <rpyOffset>0 0 0</rpyOffset>
-                    <frameName>base_link</frameName>
-                </plugin>
-                <pose>0 0 0 0 0 0</pose>
-            </sensor>
-        </gazebo>
+        <xacro:if value="$(eval sim_type=='gazebo')"/>
+            <gazebo reference="${frame}">
+                <gravity>true</gravity>
+                <sensor name="imu_sensor" type="imu">
+                    <always_on>true</always_on>
+                    <update_rate>100</update_rate>
+                    <visualize>true</visualize>
+                    <topic>${topic}</topic>
+                    <plugin filename="libgazebo_ros_imu_sensor.so" name="imu_plugin">
+                        <topicName>${topic}</topicName>
+                        <bodyName>${frame}</bodyName>
+                        <updateRateHZ>${update_rate}</updateRateHZ>
+                        <gaussianNoise>0.0</gaussianNoise>
+                        <xyzOffset>0 0 0</xyzOffset>
+                        <rpyOffset>0 0 0</rpyOffset>
+                        <frameName>base_link</frameName>
+                    </plugin>
+                    <pose>0 0 0 0 0 0</pose>
+                </sensor>
+            </gazebo>
+        </xacro:if>
+        <xacro:if value="$(eval sim_type=='gz_sim')"/>
+            <gazebo reference="${frame}">
+                <gravity>true</gravity>
+                <sensor name="imu_sensor" type="imu">
+                    <always_on>true</always_on>
+                    <update_rate>100</update_rate>
+                    <visualize>true</visualize>
+                    <topic>${topic}</topic>
+                    <imu>
+                        <!-- add noise and other parameters if required -->
+                    </imu>
+                    <pose>0 0 0 0 0 0</pose>
+                </sensor>
+            </gazebo>
+        </xacro:if>
     </xacro:macro>
 </robot>

File: copernicus_sim/urdf/accessories/lidar_copernicus.urdf.xacro (robot description, xacro)
@@ -92,32 +92,52 @@
       </xacro:if>
       <gazebo reference="${frame}">
-        <sensor type="ray" name="${frame}">
-          <always_on>true</always_on>
-          <pose>0 0 0 0 0 0</pose>
-          <visualize>false</visualize>
-          <update_rate>${update_rate}</update_rate>
-          <ray>
-            <scan>
-              <horizontal>
-                <samples>${sample_size}</samples>
-                <resolution>1</resolution>
-                <min_angle>${min_angle}</min_angle>
-                <max_angle>${max_angle}</max_angle>
-              </horizontal>
-            </scan>
-            <range>
-              <min>${min_range}</min>
-              <max>${max_range}</max>
-              <resolution>0.01</resolution>
-            </range>
-          </ray>
-          <plugin name="gazebo_ros_laser" filename="libgazebo_ros_laser.so">
-            <topicName>${topic}</topicName>
-            <frameName>${frame}</frameName>
-            <robotNamespace>${robot_namespace}</robotNamespace>
-            <gaussianNoise>0.005</gaussianNoise>
-            <alwaysOn>true</alwaysOn>
-          </plugin>
-        </sensor>
+        <xacro:if value="$(eval sim_type=='gazebo')">
+          <sensor name="laser" type="ray">
+                <pose> 0 0 0 0 0 0 </pose>
+                <visualize>false</visualize>
+                <update_rate>10</update_rate>
+                <ray>
+                    <scan>
+                        <horizontal>
+                            <samples>360</samples>
+                            <min_angle>-3.14</min_angle>
+                            <max_angle>3.14</max_angle>
+                        </horizontal>
+                    </scan>
+                    <range>
+                        <min>0.3</min>
+                        <max>12</max>
+                    </range>
+                </ray>
+                <plugin name="laser_controller" filename="libgazebo_ros_ray_sensor.so">
+                    <ros>
+                        <argument>~/out:=scan</argument>
+                    </ros>
+                    <output_type>sensor_msgs/LaserScan</output_type>
+                    <frame_name>${frame}</frame_name>
+                </plugin>
+            </sensor>
+          </xacro:if>
+          <xacro:if value="$(eval sim_type=='gz_sim')">
+          <sensor name="laser" type="gpu_lidar">
+                <pose> 0 0 0 0 0 0 </pose>
+                <visualize>false</visualize>
+                <update_rate>10</update_rate>
+                <lidar>
+                    <scan>
+                        <horizontal>
+                            <samples>360</samples>
+                            <min_angle>-3.14</min_angle>
+                            <max_angle>3.14</max_angle>
+                        </horizontal>
+                    </scan>
+                    <range>
+                        <min>0.3</min>
+                        <max>12</max>
+                    </range>
+                </lidar>
+                <topic>/model/copernicus/scan</topic>
+            </sensor>
+          </xacro:if>
       </gazebo>
   </xacro:macro>

File: copernicus_sim/urdf/components/sensors.urdf.xacro (robot description, xacro)
@@ -1,5 +1,4 @@
 <!-- IMU -->
 <robot xmlns:xacro="http://www.ros.org/wiki/xacro">
-        <xacro:if value="$(eval sim_type == 'gazebo')">
             <xacro:if value="$(arg imu_enabled)">
                 <xacro:include filename="$(find copernicus_sim)/urdf/accessories/imu_copernicus.urdf.xacro"/>
@@ -33,15 +32,4 @@
         <!-- Add frames for each of these sensors to work in gz_sim -->
         <xacro:if value="$(eval sim_type == 'gz_sim')">
-            <!-- <gazebo reference="imu" >
-                <sensor name="imu" type="imu">
-                <always_on>1</always_on>
-                <update_rate>100</update_rate>
-                <visualize>false</visualize>
-                <topic>/model/robot/imu</topic>
-                <frame_id>imu</frame_id>
-                <gz_frame_id>imu</gz_frame_id>
-                <ign_frame_id>imu</ign_frame_id>
-                </sensor>
-            </gazebo> -->
             <!-- <gazebo reference="laser2d">
                 <sensor name="laser2d" type='gpu_lidar'>"

File: copernicus_sim/urdf/copernicus.urdf.xacro (robot description, xacro)
@@ -33,11 +33,9 @@
     <xacro:arg name="robot_namespace" default="/" />
     <xacro:arg name="lidar_enabled" default="false"/>
-    <xacro:arg name="test_lidar_enabled" default="false"/>
-    <xacro:arg name="sick_lms151_enabled" default="false"/>
+    <xacro:arg name="test_lidar_enabled" default="true"/>
+    <xacro:arg name="sick_lms151_enabled" default="true"/>
     <xacro:arg name="velodyne_enabled" default="true"/>
     <xacro:arg name="imu_enabled" default="true"/>
-    <!--<xacro:arg name="camera_enabled" default="false"/>
-    <xacro:arg name="intel_d435i_enabled" default="false"/>-->
-    <xacro:include filename="$(find copernicus_sim)/urdf/copernicus_sim_control.urdf.xacro"/>
+    <xacro:include filename="$(find copernicus_sim)/urdf/gazebo_control.xacro"/>
     <xacro:include filename="$(find copernicus_sim)/urdf/components/sensors.urdf.xacro"/>
     <xacro:macro name="copernicus_robot">
