Commit message: Package cleanup

File: copernicus_sim/urdf/accessories/imu_copernicus.urdf.xacro (robot description, xacro)
@@ -25,5 +25,5 @@
 -->
 <robot name="copernicus" xmlns:xacro="https://ros.org/wiki/xacro">
-    <xacro:macro name="imu" params="frame:=imu topic:=imu/data update_rate:=20 robot_namespace:=/ sim_type:=gazebo">
+    <xacro:macro name="imu" params="frame:=imu topic:=imu/data update_rate:=20 robot_namespace:=/">
         <joint name="${frame}_joint" type="fixed">
             <parent link="base_link" />
@@ -38,5 +38,5 @@
             </inertial>
         </link>
-        <xacro:if value="$(eval sim_type=='gazebo')"/>
+        <xacro:if value="$(eval sim_type=='gazebo')">
             <gazebo reference="${frame}">
                 <gravity>true</gravity>
@@ -59,16 +59,57 @@
             </gazebo>
         </xacro:if>
-        <xacro:if value="$(eval sim_type=='gz_sim')"/>
+        <xacro:if value="$(eval sim_type=='gz_sim')">
             <gazebo reference="${frame}">
-                <gravity>true</gravity>
                 <sensor name="imu_sensor" type="imu">
+                    <plugin filename="libignition-gazebo-imu-system.so" name="ignition::gazebo::systems::Imu">
+                        <!-- Additional IMU parameters -->
+                        <initial_orientation_as_reference>false</initial_orientation_as_reference>
+                    </plugin>
                     <always_on>true</always_on>
-                    <update_rate>100</update_rate>
+                    <topic>/model/copernicus/${topic}</topic>
+                    <update_rate>${update_rate}</update_rate>
                     <visualize>true</visualize>
-                    <topic>${topic}</topic>
                     <imu>
-                        <!-- add noise and other parameters if required -->
+                        <angular_velocity>
+                            <x>
+                                <noise type="gaussian">
+                                    <mean>0.0</mean>
+                                    <stddev>2e-4</stddev>
+                                </noise>
+                            </x>
+                            <y>
+                                <noise type="gaussian">
+                                    <mean>0.0</mean>
+                                    <stddev>2e-4</stddev>
+                                </noise>
+                            </y>
+                            <z>
+                                <noise type="gaussian">
+                                    <mean>0.0</mean>
+                                    <stddev>2e-4</stddev>
+                                </noise>
+                            </z>
+                        </angular_velocity>
+                        <linear_acceleration>
+                            <x>
+                                <noise type="gaussian">
+                                    <mean>0.0</mean>
+                                    <stddev>1.7e-2</stddev>
+                                </noise>
+                            </x>
+                            <y>
+                                <noise type="gaussian">
+                                    <mean>0.0</mean>
+                                    <stddev>1.7e-2</stddev>
+                                </noise>
+                            </y>
+                            <z>
+                                <noise type="gaussian">
+                                    <mean>0.0</mean>
+                                    <stddev>1.7e-2</stddev>
+                                </noise>
+                            </z>
+                        </linear_acceleration>
                     </imu>
-                    <pose>0 0 0 0 0 0</pose>
                 </sensor>
             </gazebo>

File: copernicus_sim/urdf/accessories/lidar_copernicus.urdf.xacro (robot description, xacro)
@@ -92,52 +92,58 @@
       </xacro:if>
       <gazebo reference="${frame}">
-        <xacro:if value="$(eval sim_type=='gazebo')">
-          <sensor name="laser" type="ray">
-                <pose> 0 0 0 0 0 0 </pose>
-                <visualize>false</visualize>
-                <update_rate>10</update_rate>
-                <ray>
-                    <scan>
-                        <horizontal>
-                            <samples>360</samples>
-                            <min_angle>-3.14</min_angle>
-                            <max_angle>3.14</max_angle>
-                        </horizontal>
-                    </scan>
-                    <range>
-                        <min>0.3</min>
-                        <max>12</max>
-                    </range>
-                </ray>
-                <plugin name="laser_controller" filename="libgazebo_ros_ray_sensor.so">
-                    <ros>
-                        <argument>~/out:=scan</argument>
-                    </ros>
-                    <output_type>sensor_msgs/LaserScan</output_type>
-                    <frame_name>${frame}</frame_name>
-                </plugin>
-            </sensor>
-          </xacro:if>
-          <xacro:if value="$(eval sim_type=='gz_sim')">
-          <sensor name="laser" type="gpu_lidar">
-                <pose> 0 0 0 0 0 0 </pose>
-                <visualize>false</visualize>
-                <update_rate>10</update_rate>
-                <lidar>
-                    <scan>
-                        <horizontal>
-                            <samples>360</samples>
-                            <min_angle>-3.14</min_angle>
-                            <max_angle>3.14</max_angle>
-                        </horizontal>
-                    </scan>
-                    <range>
-                        <min>0.3</min>
-                        <max>12</max>
-                    </range>
-                </lidar>
-                <topic>/model/copernicus/scan</topic>
-            </sensor>
-          </xacro:if>
+      <sensor name="laser" type="ray">
+            <pose> 0 0 0 0 0 0 </pose>
+            <visualize>false</visualize>
+            <update_rate>10</update_rate>
+            <ray>
+                <scan>
+                    <horizontal>
+                        <samples>360</samples>
+                        <min_angle>-3.14</min_angle>
+                        <max_angle>3.14</max_angle>
+                    </horizontal>
+                </scan>
+                <range>
+                    <min>0.3</min>
+                    <max>12</max>
+                </range>
+            </ray>
+            <plugin name="laser_controller" filename="libgazebo_ros_ray_sensor.so">
+                <ros>
+                    <argument>~/out:=scan</argument>
+                </ros>
+                <output_type>sensor_msgs/LaserScan</output_type>
+                <frame_name>${frame}</frame_name>
+            </plugin>
+        </sensor>
+        <!-- <sensor type="ray" name="${frame}">
+          <always_on>true</always_on>
+          <pose>0 0 0 0 0 0</pose>
+          <visualize>false</visualize>
+          <update_rate>${update_rate}</update_rate>
+          <ray>
+            <scan>
+              <horizontal>
+                <samples>${sample_size}</samples>
+                <resolution>1</resolution>
+                <min_angle>${min_angle}</min_angle>
+                <max_angle>${max_angle}</max_angle>
+              </horizontal>
+            </scan>
+            <range>
+              <min>${min_range}</min>
+              <max>${max_range}</max>
+              <resolution>0.01</resolution>
+            </range>
+          </ray>
+          <plugin name="gazebo_ros_laser" filename="libgazebo_ros_ray_sensor.so">
+            <ros>
+              <argument>~/out:=${robot_namespace}/${topic}</argument>
+            </ros>
+            <frame_name>${frame}</frame_name>
+            <gaussianNoise>0.005</gaussianNoise>
+            <alwaysOn>true</alwaysOn>
+          </plugin>
+        </sensor> -->
       </gazebo>
   </xacro:macro>

File: copernicus_sim/urdf/components/sensors.urdf.xacro (robot description, xacro)
@@ -1,7 +1,6 @@
-<!-- IMU -->
-<robot xmlns:xacro="http://www.ros.org/wiki/xacro">
+<robot name="copernicus" xmlns:xacro="http://www.ros.org/wiki/xacro">
             <xacro:if value="$(arg imu_enabled)">
                 <xacro:include filename="$(find copernicus_sim)/urdf/accessories/imu_copernicus.urdf.xacro"/>
-                <xacro:imu robot_namespace="$(arg robot_namespace)"></xacro:imu>
+                <xacro:imu update_rate="100" robot_namespace="$(arg robot_namespace)"></xacro:imu>
             </xacro:if>
             <!-- LIDAR -->
@@ -19,84 +18,8 @@
                 <xacro:include filename="$(find copernicus_sim)/urdf/accessories/velodyne_mount.urdf.xacro"/>
                 <xacro:velodyne_mount></xacro:velodyne_mount>
-                <xacro:include filename="$(find velodyne_description)/urdf/VLP-16.urdf.xacro"/>
-                <xacro:VLP-16 parent="velodyne_mount" name="velodyne" topic="velodyne_points" hz="10" samples="440" gpu="false" min_range="0.2">
-                    <origin xyz="${velodyne_joint_x} ${velodyne_joint_y} ${velodyne_joint_z}" rpy="0 ${-velodyne_joint_pitch} 0" />
-                </xacro:VLP-16>
+                <xacro:include filename="$(find copernicus_sim)/urdf/accessories/velodyne.urdf.xacro"/>
+                    <xacro:velodyne parent="velodyne_mount" name="velodyne" topic="velodyne_points" hz="10" samples="440" gpu="false" min_range="0.2">
+                        <origin xyz="${velodyne_joint_x} ${velodyne_joint_y} ${velodyne_joint_z}" rpy="0 ${-velodyne_joint_pitch} 0" />
+                    </xacro:velodyne>
             </xacro:if>
-            <!-- CAMERA -->
-            <!-- <xacro:if value="$(arg camera_enabled)">
-                <xacro:include filename="$(find copernicus_sim)/urdf/accessories/camera_copernicus.urdf.xacro"/>
-                <xacro:camera_ intel_d435i_enabled="$(arg intel_d435i_enabled)" robot_namespace="$(arg robot_namespace)"></xacro:camera_>
-            </xacro:if> -->
-        </xacro:if>
-        <!-- Add frames for each of these sensors to work in gz_sim -->
-        <xacro:if value="$(eval sim_type == 'gz_sim')">
-            <!-- <gazebo reference="laser2d">
-                <sensor name="laser2d" type='gpu_lidar'>"
-                <pose relative_to='laser2d'>0 0 0 0 0 0</pose>
-                <topic>/model/robot/scan</topic>
-                <update_rate>10</update_rate>
-                <ray>
-                    <scan>
-                    <horizontal>
-                        <samples>270</samples>
-                        <resolution>1</resolution>
-                        <min_angle>-2.356194</min_angle>
-                        <max_angle> 2.356194</max_angle>
-                    </horizontal>
-                    <vertical>
-                        <samples>1</samples>
-                        <resolution>0.01</resolution>
-                        <min_angle>0</min_angle>
-                        <max_angle>0</max_angle>
-                    </vertical>
-                    </scan>
-                    <range>
-                        <min>0.08</min>
-                        <max>15.0</max>
-                        <resolution>0.01</resolution>
-                    </range>
-                </ray>
-                <always_on>1</always_on>
-                <visualize>true</visualize>
-                <frame_id>laser2d</frame_id>
-                <gz_frame_id>laser2d</gz_frame_id>
-                <ign_frame_id>laser2d</ign_frame_id>
-                </sensor>
-            </gazebo> -->
-<!--
-            <gazebo reference="laser3d">
-                <sensor name="laser3d" type='gpu_lidar'>"
-                <pose relative_to='laser3d'>0 0 0 0 0 0</pose>
-                <topic>/model/robot/cloud</topic>
-                <update_rate>10</update_rate>
-                <ray>
-                    <scan>
-                    <horizontal>
-                        <samples>128</samples>
-                        <resolution>0.01</resolution>
-                        <min_angle>${-M_PI}</min_angle>
-                        <max_angle>${M_PI}</max_angle>
-                    </horizontal>
-                    <vertical>
-                        <samples>32</samples>
-                        <resolution>0.01</resolution>
-                        <min_angle>${-M_PI / 16.0}</min_angle>
-                        <max_angle>${M_PI / 4.0}</max_angle>
-                    </vertical>
-                    </scan>
-                    <range>
-                        <min>0.2</min>
-                        <max>100.0</max>
-                        <resolution>0.01</resolution>
-                    </range>
-                </ray>
-                <always_on>1</always_on>
-                <visualize>true</visualize>
-                <frame_id>laser3d</frame_id>
-                <gz_frame_id>laser3d</gz_frame_id>
-                <ign_frame_id>laser3d</ign_frame_id>
-                </sensor>
-            </gazebo> -->
-        </xacro:if>
 </robot>

File: copernicus_sim/urdf/copernicus.urdf.xacro (robot description, xacro)
@@ -30,11 +30,12 @@
     <!-- xacro properties -->
     <xacro:property name="PI" value="3.14159"/>
+    <xacro:property name="M_PI" value="3.14159"/>
     <!-- xacro args -->
     <xacro:arg name="robot_namespace" default="/" />
     <xacro:arg name="lidar_enabled" default="false"/>
-    <xacro:arg name="test_lidar_enabled" default="true"/>
-    <xacro:arg name="sick_lms151_enabled" default="true"/>
-    <xacro:arg name="velodyne_enabled" default="true"/>
-    <xacro:arg name="imu_enabled" default="true"/>
+    <xacro:arg name="test_lidar_enabled" default="false"/>
+    <xacro:arg name="sick_lms151_enabled" default="false"/>
+    <xacro:arg name="velodyne_enabled" default="false"/>
+    <xacro:arg name="imu_enabled" default="false"/>
     <xacro:include filename="$(find copernicus_sim)/urdf/gazebo_control.xacro"/>
     <xacro:include filename="$(find copernicus_sim)/urdf/components/sensors.urdf.xacro"/>

File: copernicus_sim/urdf/gazebo_control.xacro (robot description, xacro)
@@ -1,69 +1,65 @@
 <?xml version="1.0"?>
 <robot xmlns:xacro="http://ros.org/wiki/xacro">
-    <!-- <link name="map"/>
-    <joint name="world_joint" type="fixed">
-        <parent link="world"/>
-        <child link="map"/>
-        <origin xyz="0 0 0" rpy="0 0 0"/>
-    </joint> -->
     <gazebo>
-            <xacro:if value="$(eval sim_type == 'gz_sim')">
-                 <plugin filename="gz-sim-diff-drive-system" name="gz::sim::systems::DiffDrive">
-                    <odom_publisher_frequency>50</odom_publisher_frequency>
-                    <left_joint>front_left_wheel_joint</left_joint>
-                    <left_joint>back_left_wheel_joint</left_joint>
-                    <right_joint>front_right_wheel_joint</right_joint>
-                    <right_joint>back_right_wheel_joint</right_joint>
-                    <wheel_separation>${base_w}</wheel_separation>
-                    <wheel_diameter>${2*wheel_radius}</wheel_diameter>
-                    <max_wheel_torque>20</max_wheel_torque>
-                    <max_linear_acceleration>1.0</max_linear_acceleration>
-                    <topic>cmd_vel</topic>
-                    <publish_odom>true</publish_odom>
-                    <publish_odom_tf>true</publish_odom_tf>
-                    <publish_wheel_tf>true</publish_wheel_tf>
-                    <odom_topic>/model/robot/odom</odom_topic>
-                    <frame_id>odom</frame_id>
-                    <child_frame_id>base_link</child_frame_id>
-                </plugin>
-                <plugin filename="gz-sim-joint-state-publisher-system" name="gz::sim::systems::JointStatePublisher">
+        <xacro:if value="$(eval sim_type == 'gz_sim')">
+                <plugin filename="gz-sim-diff-drive-system" name="gz::sim::systems::DiffDrive">
+                <odom_publisher_frequency>100</odom_publisher_frequency>
+                <left_joint>front_left_wheel_joint</left_joint>
+                <left_joint>back_left_wheel_joint</left_joint>
+                <right_joint>front_right_wheel_joint</right_joint>
+                <right_joint>back_right_wheel_joint</right_joint>
+                <wheel_separation>${base_w}</wheel_separation>
+                <wheel_diameter>${2*wheel_radius}</wheel_diameter>
+                <max_wheel_torque>20</max_wheel_torque>
+                <max_linear_acceleration>1.0</max_linear_acceleration>
+                <topic>cmd_vel</topic>
+                <publish_odom>true</publish_odom>
+                <publish_odom_tf>true</publish_odom_tf>
+                <publish_wheel_tf>true</publish_wheel_tf>
+                <tf_topic>/model/copernicus/tf_odom</tf_topic>
+                <odom_topic>/model/copernicus/odom</odom_topic>
+                <frame_id>odom</frame_id>
+                <child_frame_id>base_link</child_frame_id>
+            </plugin>
+            <plugin filename="gz-sim-joint-state-publisher-system" name="gz::sim::systems::JointStatePublisher">
+                <update_rate>100</update_rate>
+                <topic>/model/copernicus/joint_states</topic>
+                <joint_name>front_left_wheel_joint</joint_name>
+                <joint_name>front_right_wheel_joint</joint_name>
+                <joint_name>back_left_wheel_joint</joint_name>
+                <joint_name>back_right_wheel_joint</joint_name>
+            </plugin>
+            <!-- Testing required -->
+            <plugin filename="gz-sim-pose-publisher-system" name="gz::sim::systems::PosePublisher">
+                <publish_link_pose>false</publish_link_pose>
+                <publish_sensor_pose>false</publish_sensor_pose>
+                <publish_model_pose>true</publish_model_pose>
+                <publish_collision_pose>false</publish_collision_pose>
+                <update_frequency>40</update_frequency>
+            </plugin>
+        </xacro:if>
+        <xacro:if value="$(eval sim_type == 'gazebo')">
+            <plugin name="differential_drive_controller" filename="libgazebo_ros_diff_drive.so">
+                <!-- Plugin update rate in Hz -->
+                <update_rate>100</update_rate>
+                <num_wheel_pairs>2</num_wheel_pairs>
+                <left_joint>front_left_wheel_joint</left_joint>
+                <right_joint>front_right_wheel_joint</right_joint>
+                <left_joint>back_left_wheel_joint</left_joint>
+                <right_joint>back_right_wheel_joint</right_joint>
+                <wheel_separation>${base_w}</wheel_separation>
+                <wheel_diameter>${2*wheel_radius}</wheel_diameter>
+                <max_wheel_torque>20</max_wheel_torque>
+                <max_wheel_acceleration>1.0</max_wheel_acceleration>
+                <frame_id>odom</frame_id>
+                <child_frame_id>base_link</child_frame_id>
+                <publish_odom>true</publish_odom>
+                <publish_odom_tf>true</publish_odom_tf>
+                <publish_wheel_tf>true</publish_wheel_tf>
+                <odometry_source>1</odometry_source>
+            </plugin>
+                <plugin name="ground_truth_publisher" filename="libgazebo_ros_p3d.so">
                     <update_rate>50</update_rate>
-                    <topic>/model/robot/joint_states</topic>
-                    <joint_name>front_left_wheel_joint</joint_name>
-                    <joint_name>front_right_wheel_joint</joint_name>
-                    <joint_name>back_left_wheel_joint</joint_name>
-                    <joint_name>back_right_wheel_joint</joint_name>
-                </plugin>
-            </xacro:if>
-            <xacro:if value="$(eval sim_type == 'gazebo')">
-                <plugin name="differential_drive_controller" filename="libgazebo_ros_diff_drive.so">
-                    <!-- Plugin update rate in Hz -->
-                    <updateRate>100</updateRate>
-                    <num_wheel_pairs>2</num_wheel_pairs>
-                    <!-- Name of left joint, defaults to `left_joint` -->
-                    <left_joint>front_left_wheel_joint</left_joint>
-                    <left_joint>back_left_wheel_joint</left_joint>
-                    <!-- Name of right joint, defaults to `right_joint` -->
-                    <right_joint>front_right_wheel_joint</right_joint>
-                    <right_joint>back_right_wheel_joint</right_joint>
-    <!-- The distance from the center of one wheel to the other, in meters, defaults to 0.34 m -->
-                    <wheel_separation>${base_w}</wheel_separation>
-                    <!-- Diameter of the wheels, in meters, defaults to 0.15 m -->
-                    <wheel_diameter>${2*wheel_radius}</wheel_diameter>
-                    <!-- Wheel acceleration, in rad/s^2, defaults to 0.0 rad/s^2 -->>
-                    <!-- Limits -->
-                    <max_wheel_torque>20</max_wheel_torque>
-                    <max_wheel_acceleration>1.0</max_wheel_acceleration>
-                    <!-- Output -->
-                    <odometry_frame>odom</odometry_frame>
-                    <robot_base_frame>base_link</robot_base_frame>
-                    <publish_odom>true</publish_odom>
-                    <publish_odom_tf>true</publish_odom_tf>
-                    <publish_wheel_tf>true</publish_wheel_tf>
-                    <odometry_source>1</odometry_source>
-                </plugin>
-                <!-- <plugin name="ground_truth_publisher" filename="libgazebo_ros_p3d.so">
-                    <update_rate>50</update_rate>
-                    <odom_topic>odom</odom_topic>
+                    <odom_topic>/copernicus/odom</odom_topic>
                     <frame_name>map</frame_name>
                     <body_name>base_link</body_name>
@@ -71,6 +67,6 @@
                     <xyz_offsets>0 0 0</xyz_offsets>
                     <rpy_offsets>0 0 0</rpy_offsets>
-                </plugin> -->
-            </xacro:if>
-        </gazebo>
+                </plugin>
+        </xacro:if>
+    </gazebo>
 </robot>
